Commit message: add navigation mapping setup and motor safety gate

File: src/helper_description/urdf/helper_robot.urdf.xacro (robot description, xacro)
@@ -1,4 +1,77 @@
 <?xml version="1.0"?>
 <robot name="helper_robot" xmlns:xacro="http://www.ros.org/wiki/xacro">
+  <xacro:property name="wheel_radius" value="0.065"/>
+  <xacro:property name="wheel_width" value="0.03"/>
+  <xacro:property name="track_width" value="0.400"/>
+  <xacro:property name="base_length" value="0.40"/>
+  <xacro:property name="base_width" value="0.30"/>
+  <xacro:property name="base_height" value="0.12"/>
+  <xacro:property name="base_mass" value="12.0"/>
+  <xacro:property name="wheel_mass" value="0.6"/>
+  <xacro:property name="sensor_mass" value="0.15"/>
+  <xacro:property name="camera_mass" value="0.1"/>
+  <xacro:property name="caster_mass" value="0.2"/>
+  <xacro:macro name="box_inertial" params="mass x y z">
+    <inertial>
+      <origin xyz="0 0 0" rpy="0 0 0"/>
+      <mass value="${mass}"/>
+      <inertia
+        ixx="${mass * (y * y + z * z) / 12.0}"
+        ixy="0"
+        ixz="0"
+        iyy="${mass * (x * x + z * z) / 12.0}"
+        iyz="0"
+        izz="${mass * (x * x + y * y) / 12.0}"/>
+    </inertial>
+  </xacro:macro>
+  <xacro:macro name="cylinder_inertial_y" params="mass radius length">
+    <inertial>
+      <origin xyz="0 0 0" rpy="0 0 0"/>
+      <mass value="${mass}"/>
+      <inertia
+        ixx="${mass * (3.0 * radius * radius + length * length) / 12.0}"
+        ixy="0"
+        ixz="0"
+        iyy="${mass * radius * radius / 2.0}"
+        iyz="0"
+        izz="${mass * (3.0 * radius * radius + length * length) / 12.0}"/>
+    </inertial>
+  </xacro:macro>
+  <xacro:macro name="cylinder_inertial_z" params="mass radius length">
+    <inertial>
+      <origin xyz="0 0 0" rpy="0 0 0"/>
+      <mass value="${mass}"/>
+      <inertia
+        ixx="${mass * (3.0 * radius * radius + length * length) / 12.0}"
+        ixy="0"
+        ixz="0"
+        iyy="${mass * (3.0 * radius * radius + length * length) / 12.0}"
+        iyz="0"
+        izz="${mass * radius * radius / 2.0}"/>
+    </inertial>
+  </xacro:macro>
+  <xacro:macro name="drive_wheel" params="side y">
+    <link name="${side}_wheel">
+      <visual>
+        <origin xyz="0 0 0" rpy="${pi / 2.0} 0 0"/>
+        <geometry>
+          <cylinder radius="${wheel_radius}" length="${wheel_width}"/>
+        </geometry>
+      </visual>
+      <collision>
+        <origin xyz="0 0 0" rpy="${pi / 2.0} 0 0"/>
+        <geometry>
+          <cylinder radius="${wheel_radius}" length="${wheel_width}"/>
+        </geometry>
+      </collision>
+      <xacro:cylinder_inertial_y mass="${wheel_mass}" radius="${wheel_radius}" length="${wheel_width}"/>
+    </link>
+    <joint name="${side}_wheel_joint" type="continuous">
+      <parent link="base_link"/>
+      <child link="${side}_wheel"/>
+      <origin xyz="0 ${y} ${wheel_radius}" rpy="0 0 0"/>
+      <axis xyz="0 1 0"/>
+    </joint>
+  </xacro:macro>
   <!-- base_link: 전륜 좌우 구동바퀴 중심 중간점 -->
   <link name="base_link">
@@ -6,35 +79,39 @@
       <origin xyz="-0.12 0 0.08" rpy="0 0 0"/>
       <geometry>
-        <box size="0.40 0.30 0.12"/>
+        <box size="${base_length} ${base_width} ${base_height}"/>
       </geometry>
     </visual>
+    <collision>
+      <origin xyz="-0.12 0 0.08" rpy="0 0 0"/>
+      <geometry>
+        <box size="${base_length} ${base_width} ${base_height}"/>
+      </geometry>
+    </collision>
+    <xacro:box_inertial mass="${base_mass}" x="${base_length}" y="${base_width}" z="${base_height}"/>
   </link>
-  <!-- left wheel -->
-  <link name="left_wheel">
+  <xacro:drive_wheel side="left" y="${track_width / 2.0}"/>
+  <xacro:drive_wheel side="right" y="${-track_width / 2.0}"/>
+  <!-- rear caster -->
+  <link name="rear_caster">
     <visual>
-      <origin xyz="0 0 0" rpy="1.5708 0 0"/>
       <geometry>
-        <cylinder radius="0.05" length="0.03"/>
+        <sphere radius="0.025"/>
       </geometry>
     </visual>
+    <collision>
+      <geometry>
+        <sphere radius="0.025"/>
+      </geometry>
+    </collision>
+    <inertial>
+      <origin xyz="0 0 0" rpy="0 0 0"/>
+      <mass value="${caster_mass}"/>
+      <inertia ixx="0.00005" ixy="0" ixz="0" iyy="0.00005" iyz="0" izz="0.00005"/>
+    </inertial>
   </link>
-  <joint name="left_wheel_joint" type="fixed">
+  <joint name="rear_caster_joint" type="fixed">
     <parent link="base_link"/>
-    <child link="left_wheel"/>
-    <origin xyz="0 0.15 0" rpy="0 0 0"/>
-  </joint>
-  <!-- right wheel -->
-  <link name="right_wheel">
-    <visual>
-      <origin xyz="0 0 0" rpy="1.5708 0 0"/>
-      <geometry>
-        <cylinder radius="0.05" length="0.03"/>
-      </geometry>
-    </visual>
-  </link>
-  <joint name="right_wheel_joint" type="fixed">
-    <parent link="base_link"/>
-    <child link="right_wheel"/>
-    <origin xyz="0 -0.15 0" rpy="0 0 0"/>
+    <child link="rear_caster"/>
+    <origin xyz="-0.28 0 0.025" rpy="0 0 0"/>
   </joint>
   <!-- front lidar -->
@@ -45,4 +122,10 @@
       </geometry>
     </visual>
+    <collision>
+      <geometry>
+        <cylinder radius="0.04" length="0.03"/>
+      </geometry>
+    </collision>
+    <xacro:cylinder_inertial_z mass="${sensor_mass}" radius="0.04" length="0.03"/>
   </link>
   <joint name="laser_front_joint" type="fixed">
@@ -58,4 +141,10 @@
       </geometry>
     </visual>
+    <collision>
+      <geometry>
+        <cylinder radius="0.04" length="0.03"/>
+      </geometry>
+    </collision>
+    <xacro:cylinder_inertial_z mass="${sensor_mass}" radius="0.04" length="0.03"/>
   </link>
   <joint name="laser_rear_joint" type="fixed">
@@ -71,4 +160,10 @@
       </geometry>
     </visual>
+    <collision>
+      <geometry>
+        <box size="0.06 0.03 0.03"/>
+      </geometry>
+    </collision>
+    <xacro:box_inertial mass="${camera_mass}" x="0.06" y="0.03" z="0.03"/>
   </link>
   <joint name="depth_camera_joint" type="fixed">
@@ -78,5 +173,5 @@
   </joint>
   <!-- rgb webcam -->
-  <link name="rgb_camera_link">
+  <!-- <link name="rgb_camera_link">
     <visual>
       <geometry>
@@ -84,9 +179,9 @@
       </geometry>
     </visual>
-  </link>
-  <joint name="rgb_camera_joint" type="fixed">
+  </link> -->
+  <!-- <joint name="rgb_camera_joint" type="fixed">
     <parent link="base_link"/>
     <child link="rgb_camera_link"/>
     <origin xyz="0.10 0 0.38" rpy="0 0 0"/>
-  </joint>
+  </joint> -->
 </robot>

Commit message: update urdf

File: src/helper_description/urdf/helper_robot.urdf.xacro (robot description, xacro)
@@ -4,12 +4,11 @@
   <xacro:property name="wheel_width" value="0.03"/>
   <xacro:property name="track_width" value="0.400"/>
-  <xacro:property name="base_length" value="0.40"/>
-  <xacro:property name="base_width" value="0.30"/>
-  <xacro:property name="base_height" value="0.12"/>
+  <xacro:property name="base_length" value="0.400"/>
+  <xacro:property name="base_width" value="0.320"/>
+  <xacro:property name="base_height" value="0.330"/>
   <xacro:property name="base_mass" value="12.0"/>
   <xacro:property name="wheel_mass" value="0.6"/>
   <xacro:property name="sensor_mass" value="0.15"/>
   <xacro:property name="camera_mass" value="0.1"/>
-  <xacro:property name="caster_mass" value="0.2"/>
   <xacro:macro name="box_inertial" params="mass x y z">
     <inertial>
@@ -77,5 +76,5 @@
   <link name="base_link">
     <visual>
-      <origin xyz="-0.12 0 0.08" rpy="0 0 0"/>
+      <origin xyz="-0.2 0 0.265" rpy="0 0 0"/>
       <geometry>
         <box size="${base_length} ${base_width} ${base_height}"/>
@@ -83,5 +82,5 @@
     </visual>
     <collision>
-      <origin xyz="-0.12 0 0.08" rpy="0 0 0"/>
+      <origin xyz="-0.2 0 0.265" rpy="0 0 0"/>
       <geometry>
         <box size="${base_length} ${base_width} ${base_height}"/>
@@ -92,27 +91,4 @@
   <xacro:drive_wheel side="left" y="${track_width / 2.0}"/>
   <xacro:drive_wheel side="right" y="${-track_width / 2.0}"/>
-  <!-- rear caster -->
-  <link name="rear_caster">
-    <visual>
-      <geometry>
-        <sphere radius="0.025"/>
-      </geometry>
-    </visual>
-    <collision>
-      <geometry>
-        <sphere radius="0.025"/>
-      </geometry>
-    </collision>
-    <inertial>
-      <origin xyz="0 0 0" rpy="0 0 0"/>
-      <mass value="${caster_mass}"/>
-      <inertia ixx="0.00005" ixy="0" ixz="0" iyy="0.00005" iyz="0" izz="0.00005"/>
-    </inertial>
-  </link>
-  <joint name="rear_caster_joint" type="fixed">
-    <parent link="base_link"/>
-    <child link="rear_caster"/>
-    <origin xyz="-0.28 0 0.025" rpy="0 0 0"/>
-  </joint>
   <!-- front lidar -->
   <link name="laser_front">
@@ -132,5 +108,5 @@
     <parent link="base_link"/>
     <child link="laser_front"/>
-    <origin xyz="0.12 0 0.18" rpy="0 0 0"/>
+    <origin xyz="0.149 0 0.2772" rpy="0 0 0"/>
   </joint>
   <!-- rear lidar -->
@@ -151,5 +127,5 @@
     <parent link="base_link"/>
     <child link="laser_rear"/>
-    <origin xyz="-0.25 0 0.18" rpy="0 0 3.14159"/>
+    <origin xyz="-0.149 0 0.2772" rpy="0 0 3.14159"/>
   </joint>
   <!-- depth camera -->
@@ -170,5 +146,5 @@
     <parent link="base_link"/>
     <child link="depth_camera_link"/>
-    <origin xyz="0.10 0 0.35" rpy="0 0 0"/>
+    <origin xyz="0.1847 0 0.1889" rpy="0 0.95993 0"/>
   </joint>
   <!-- rgb webcam -->

Commit message: update urdf

File: src/helper_description/urdf/helper_robot.urdf.xacro (robot description, xacro)
@@ -108,5 +108,5 @@
     <parent link="base_link"/>
     <child link="laser_front"/>
-    <origin xyz="0.149 0 0.2772" rpy="0 0 0"/>
+    <origin xyz="0.149 0 0.2772" rpy="0 0 3.14159"/>
   </joint>
   <!-- rear lidar -->

Commit message: update perception&navigation logic

File: src/helper_description/urdf/helper_robot.urdf.xacro (robot description, xacro)
@@ -148,4 +148,11 @@
     <origin xyz="0.1847 0 0.1889" rpy="0 0.95993 0"/>
   </joint>
+  <!-- Attach the depth-camera driver's TF tree at its camera_link root. -->
+  <link name="camera_link"/>
+  <joint name="depth_camera_driver_joint" type="fixed">
+    <parent link="depth_camera_link"/>
+    <child link="camera_link"/>
+    <origin xyz="0 0 0" rpy="0 0 0"/>
+  </joint>
   <!-- rgb webcam -->
   <!-- <link name="rgb_camera_link">

Commit message: update percepetion & navgiation

File: src/helper_description/urdf/helper_robot.urdf.xacro (robot description, xacro)
@@ -146,5 +146,5 @@
     <parent link="base_link"/>
     <child link="depth_camera_link"/>
-    <origin xyz="0.1847 0 0.1889" rpy="0 0.95993 0"/>
+    <origin xyz="0.1847 0 0.1889" rpy="0 0 0"/>
   </joint>
   <!-- Attach the depth-camera driver's TF tree at its camera_link root. -->
